File: KiCad/BusinessCard/BusinessCard.kicad_sch (KiCad schematic)
At the start: 0 parts

Commit message: KiCad chematic ready without values or footprints.
Parts:
- added C1: C, symbol Device:C
- added D1, D2: D_Zener, symbol Device:D_Zener
- added D3: LED, symbol Device:LED
- added R1, R2: 68R, symbol Device:R
- added R3: R, symbol Device:R
- added R4: 330R, symbol Device:R
- added U1: ATtiny85-20P, Package_DIP:DIP-8_W7.62mm, symbol MCU_Microchip_ATtiny:ATtiny85-20P
- added U2: (no value), symbol #custom_library:PCB_USB_connector
Connections:
- new net: D3.1 (K), R4.2
- new net: D2.1 (K), R2.2, U2.3 (D+)
- new net: R2.1, U1.3 (XTAL2/PB4)
- new net: R1.1, U1.2 (XTAL1/PB3)
- new net: D3.2 (A), U1.6 (PB1)
- new net: D1.1 (K), R1.2, R3.2, U2.2 (D-)
- new net GND: C1.2, D1.2 (A), D2.2 (A), R4.1, U1.4 (GND), U2.4 (GND)
- new net VCC: C1.1, R3.1, U1.8 (VCC), U2.1 (Vcc)
